Commit message: Added test for collision interface, passed

File: test/test_models/meldog_base_link.urdf (robot description, URDF)
Before this commit: robot meldog_core, 18 links, 17 joints
Links:
- link LFF_link: geometry collision sphere radius=0.1
- link LFLL_link: geometry collision sphere radius=0.1
- link LRF_link: geometry collision sphere radius=0.1
- link LRLL_link: geometry collision sphere radius=0.5
- link RFF_link: geometry collision sphere radius=0.1
- link RFLL_link: geometry collision sphere radius=1.0
- link RRF_link: geometry collision sphere radius=0.1
- link RRLL_link: geometry collision cylinder length=1.5 radius=0.

Commit message: New stable run in demo

File: test/test_models/meldog_base_link.urdf (robot description, URDF)
Before this commit: robot meldog_core, 18 links, 17 joints
Joints:
- joint LFH_joint: limit lower=-120 upper=120 effort=34.895 velocity=18.906274745776084 -> lower=-1.57 upper=0.0 effort=34.895 velocity=18.906274745776084
- joint LRH_joint: limit lower=-120 upper=120 effort=34.895 velocity=18.906274745776084 -> lower=-1.57 upper=0.0 effort=34.895 velocity=18.906274745776084
- joint RFH_joint: limit lower=-120 upper=120 effort=34.895 velocity=18.906274745776084 -> lower=-1.57 upper=0.0 effort=34.895 velocity=18.906274745776084
- joint RRH_joint: limit lower=-120 upper=120 effort=34.895 velocity=18.906274745776084 -> lower=-1.57 upper=0.0 effort=34.895 velocity=18.906274745776084
