Commit message: Im done with Melman for now

File: test/test_models/melman.urdf (robot description, URDF)
Before this commit: robot Melman, 26 links, 25 joints
Links:
- link Left_ArmMounting: geometry collision sphere radius=0.022
- link Right_ArmMounting: geometry collision sphere radius=0.022
- link Trunk: geometry collision sphere radius=0.048; collision sphere radius=0.048
